Commit message: Adding files

File: src/hri_control/models/shadow_hand_right.urdf (robot description, URDF)
Before this commit: robot shadow_right, 33 links, 32 joints
Links:
- link forearm: geometry collision box size=0.07 0.07 0.07; collision mesh filename=meshes/collision/forearm_E3M5.obj scale=0.001 0.001 0.001
